Commit message: added control for prototype and basic environment

File: src/tfr_description/xacro/proto_constants.xacro (robot description, xacro)
@@ -5,5 +5,5 @@
   <xacro:property name="base_length" value="${58*itom}"/> <!-- Max val: 50" bare minimum -->
   <xacro:property name="base_height" value="${2*itom}"/>
-  <xacro:property name="base_mass"   value="5"
+  <xacro:property name="base_mass"   value="5"/>
   <xacro:property name="wheel_radius" value="${6*itom}"/>
   <xacro:property name="wheel_width" value="${6*itom}"/>

File: src/tfr_description/xacro/proto_drivebase_controller.xacro (robot description, xacro)
@@ -31,5 +31,5 @@
       <wheelDiameter>${wheel_radius*2}</wheelDiameter>
       <robotBaseFrame>god</robotBaseFrame>
-      <torque>10</torque>
+      <torque>20</torque>
       <topicName>cmd_vel</topicName>
       <commandTopic>cmd_vel</commandTopic>

File: src/tfr_description/xacro/proto_model.xacro (robot description, xacro)
@@ -62,5 +62,5 @@
     <inertial>
       <mass value="${base_mass}"/>
-      <inertia ixx="${base_mass/12*(base_width**2+base_depth**2)}" ixy="0.0" ixz="0.0" iyy="${base_mass/12*(base_depth**2+base_height**2)}" iyz="0.0" izz="${base_mass/12*(base_width**2+base_height**2)}"/>
+      <inertia ixx="${base_mass/12*(base_width**2+base_length**2)}" ixy="0.0" ixz="0.0" iyy="${base_mass/12*(base_length**2+base_height**2)}" iyz="0.0" izz="${base_mass/12*(base_width**2+base_height**2)}"/>
     </inertial>
   </link>
