Commit message: Various cleanup bits
Cleaned up lots of package.xml's, removed the unnecessary echo node,
fixed some XML formatting inconsistencies, and made all the PID values
equal to {1.0, 500.0, 0.0} for now since we have no way to test them.

File: src/tfr_description/xacro/model.xacro (robot description, xacro)
@@ -1,5 +1,5 @@
 <?xml version="1.0"?>
 <robot name="excavator" xmlns:xacro="http://www.ros.org/wiki/xacro">
-  <!--top level robot description-->
+  <!-- Top-level robot description -->
   <xacro:include filename="model_constants.xacro"/>
   <xacro:include filename="model_base.xacro"/>

File: src/tfr_description/xacro/model_arm.xacro (robot description, xacro)
@@ -21,5 +21,5 @@
     <origin xyz="${base_length/2-base_width/3-3*itom} 0 ${base_height/2}" />
     <axis xyz="0 0 1" />
-    <limit effort="1.0" velocity="1.0"/>
+    <limit effort="1.0" velocity="1.0" />
   </joint>
   <transmission name="turntable_tran">
@@ -53,5 +53,5 @@
     <axis xyz="0 1 0" />
     <origin xyz="${turntable_radius} 0 ${turntable_height}" />
-    <limit effort="1.0" velocity="1.0" lower="${lower_arm_min}" upper="${lower_arm_max}"/>
+    <limit effort="1.0" velocity="1.0" lower="${lower_arm_min}" upper="${lower_arm_max}" />
   </joint>
   <transmission name="lower_arm_tran">
@@ -85,5 +85,5 @@
     <axis xyz="0 1 0" />
     <origin xyz="0 0 ${lower_arm_length}" />
-    <limit effort="1.0" velocity="1.0" lower="${upper_arm_min}" upper="${upper_arm_max}"/>
+    <limit effort="1.0" velocity="1.0" lower="${upper_arm_min}" upper="${upper_arm_max}" />
   </joint>
   <transmission name="upper_arm_tran">

File: src/tfr_description/xacro/model_base.xacro (robot description, xacro)
@@ -1,6 +1,19 @@
 <?xml version="1.0"?>
 <robot xmlns:xacro="http://www.ros.org/wiki/xacro" name="excavator">
-  <!--DRIVEBASE-->
-  <!-- A macro for creating a wheel with a link, joint, and transmission -->
+  <!-- CHASSIS -->
+  <link name="base_link" >
+    <visual>
+      <geometry>
+        <box size="${base_length} ${base_width} ${base_height}" />
+      </geometry>
+    </visual>
+    <collision>
+      <geometry>
+        <box size="${base_length} ${base_width} ${base_height}" />
+      </geometry>
+    </collision>
+  </link>
+  <!-- DRIVEBASE -->
+  <!-- A macro for creating a wheel with a link and joint -->
   <xacro:macro name="wheel" params="name fb lr">
     <link name="${name}">
@@ -19,11 +32,12 @@
     </link>
     <joint name="${name}_joint" type="continuous">
-      <parent link="base_link"/>
-      <child link="${name}"/>
-      <origin xyz="${fb*base_length/2 - fb*wheel_radius} ${lr*base_width/2 + lr*wheel_width/2} ${-base_height/2}"/>
+      <parent link="base_link" />
+      <child link="${name}" />
+      <origin xyz="${fb*base_length/2 - fb*wheel_radius} ${lr*base_width/2 + lr*wheel_width/2} ${-base_height/2}" />
       <axis xyz="0 1 0"/>
-      <limit effort="1.0"  velocity="1.0"/>
+      <limit effort="1.0" velocity="1.0" />
     </joint>
   </xacro:macro>
+  <!-- A macro for creating a wheel transmission -->
   <xacro:macro name="wheel_tran" params="name">
     <transmission name="${name}_tran">
@@ -39,26 +53,13 @@
     </transmission>
   </xacro:macro>
-  <!--stamp out the "treads" (just individual wheels) -->
+  <!-- Create the "treads" (just individual wheels) -->
   <xacro:wheel name="left_tread" fb="-1" lr="1" />
   <xacro:wheel_tran name="left_tread" />
   <xacro:wheel name="right_tread" fb = "-1" lr="-1" />
   <xacro:wheel_tran name="right_tread" />
-  <!-- add extra, free-spinning wheels so the robot doesn't wobble in simulation -->
+  <!-- Add extra free-spinning wheels for the other end of the robot -->
   <xacro:wheel name="left_tread_f" fb="1" lr="1" />
   <xacro:wheel name="right_tread_f" fb="1" lr="-1" />
-  <!--CHASSIS-->
-  <link name="base_link" >
-    <visual>
-      <geometry>
-        <box size="${base_length} ${base_width} ${base_height}" />
-      </geometry>
-    </visual>
-    <collision>
-      <geometry>
-        <box size="${base_length} ${base_width} ${base_height}" />
-      </geometry>
-    </collision>
-  </link>
-  <!--BIN-->
+  <!-- BIN -->
   <link name="bin" >
     <visual>
@@ -80,5 +81,5 @@
     <axis xyz="0 -1 0" />
     <origin xyz="${-base_length/2} 0 ${base_height/2}" />
-    <limit effort="1.0"  velocity="1.0" lower="0" upper="${pi/4}"/>
+    <limit effort="1.0" velocity="1.0" lower="0" upper="${pi/4}" />
   </joint>
 </robot>

File: src/tfr_description/xacro/model_constants.xacro (robot description, xacro)
@@ -1,40 +1,41 @@
 <?xml version="1.0"?>
 <robot name="excavator" xmlns:xacro="http://www.ros.org/wiki/xacro">
-  <!--shared model level constants-->
-  <xacro:property name="itom" value="0.0254"/> <!-- Inches to meters conversion -->
-  <xacro:property name="dtor" value="${pi/180}"/> <!-- Degrees to radians conversion -->
-  <!--drivebase parameters-->
-  <xacro:property name="base_width" value="${20*itom}"/>
-  <xacro:property name="base_length" value="${50*itom}"/>
-  <xacro:property name="base_height" value="${6*itom}"/>
-  <!--wheel parameters-->
-  <xacro:property name="wheel_radius" value="${5.5*itom}"/>
-  <xacro:property name="wheel_width" value="${5.75*itom}"/>
-  <!--bin parameters-->
+  <!-- Shared model level constants -->
+  <xacro:property name="itom" value="0.0254" /> <!-- Inches to meters conversion -->
+  <xacro:property name="dtor" value="${pi/180}" /> <!-- Degrees to radians conversion -->
+  <!-- Drivebase parameters -->
+  <xacro:property name="base_width" value="${20*itom}" />
+  <xacro:property name="base_length" value="${50*itom}" />
+  <xacro:property name="base_height" value="${6*itom}" />
+  <!-- Wheel parameters -->
+  <xacro:property name="wheel_radius" value="${5.5*itom}" />
+  <xacro:property name="wheel_width" value="${5.75*itom}" />
+  <!-- Bin parameters -->
   <!-- Length of top of bin, length of bottom is 13.86 -->
   <!-- Using the bigger size as a box instead of making a complex angled shape -->
-  <xacro:property name="bin_length" value="${25.78*itom}"/>
-  <xacro:property name="bin_width" value="${base_width}"/>
-  <xacro:property name="bin_height" value="${12*itom}"/>
-  <!--turntable parameters-->
-  <xacro:property name="turntable_radius" value="${6*itom}"/>
+  <xacro:property name="bin_length" value="${25.78*itom}" />
+  <xacro:property name="bin_width" value="${base_width}" />
+  <xacro:property name="bin_height" value="${12*itom}" />
+  <!-- Turntable parameters -->
+  <xacro:property name="turntable_radius" value="${6*itom}" />
   <!-- 1" in model plus undefined height for mounting plates and extra components -->
-  <xacro:property name="turntable_height" value="${2*itom}"/>
-  <!--lower arm parameters-->
-  <xacro:property name="lower_arm_length" value="${22*itom}"/>
-  <xacro:property name="lower_arm_width" value="${4*itom}"/>
-  <xacro:property name="lower_arm_height" value="${3.5*itom}"/>
-  <xacro:property name="lower_arm_min" value="${11.74*dtor}"/>
-  <xacro:property name="lower_arm_max" value="${97*dtor}"/>
-  <!--upper arm parameters-->
-  <xacro:property name="upper_arm_length" value="${20*itom}"/>
-  <xacro:property name="upper_arm_width" value="${3.61*itom}"/>
-  <xacro:property name="upper_arm_height" value="${2.5*itom}"/>
-  <xacro:property name="upper_arm_min" value="${0*dtor}"/>
-  <xacro:property name="upper_arm_max" value="${107*dtor}"/>
-  <!--scoop parameters-->
-  <xacro:property name="scoop_width" value="${10*itom}"/>
-  <xacro:property name="scoop_diameter" value="${10.75*itom}"/>
-  <xacro:property name="scoop_min" value="${-50*dtor}"/>
-  <xacro:property name="scoop_max" value="${65*dtor}"/>
+  <!-- Rounded to 2" for now -->
+  <xacro:property name="turntable_height" value="${2*itom}" />
+  <!-- Lower arm parameters -->
+  <xacro:property name="lower_arm_length" value="${22*itom}" />
+  <xacro:property name="lower_arm_width" value="${4*itom}" />
+  <xacro:property name="lower_arm_height" value="${3.5*itom}" />
+  <xacro:property name="lower_arm_min" value="${11.74*dtor}" />
+  <xacro:property name="lower_arm_max" value="${97*dtor}" />
+  <!-- Upper arm parameters -->
+  <xacro:property name="upper_arm_length" value="${20*itom}" />
+  <xacro:property name="upper_arm_width" value="${3.61*itom}" />
+  <xacro:property name="upper_arm_height" value="${2.5*itom}" />
+  <xacro:property name="upper_arm_min" value="${0*dtor}" />
+  <xacro:property name="upper_arm_max" value="${107*dtor}" />
+  <!-- Scoop parameters -->
+  <xacro:property name="scoop_width" value="${10*itom}" />
+  <xacro:property name="scoop_diameter" value="${10.75*itom}" />
+  <xacro:property name="scoop_min" value="${-50*dtor}" />
+  <xacro:property name="scoop_max" value="${65*dtor}" />
 </robot>
