Commit message: Fixed all the model dimensions that I could
Also removed all physical properties for now as they're much harder to
pin down and after a recent discovery I made we may not be using Gazebo
at all, which makes the physical properties irrelevant and just a waste
of space.

File: src/tfr_description/xacro/model_arm.xacro (robot description, xacro)
@@ -5,18 +5,14 @@
     <visual>
       <geometry>
-        <cylinder radius="${base_width/3}" length="${6*itom}" />
+        <cylinder radius="${turntable_radius}" length="${turntable_height}" />
       </geometry>
-      <origin xyz="0 0 ${3*itom}" />
+      <origin xyz="0 0 ${turntable_height/2}" />
     </visual>
     <collision>
       <geometry>
-        <cylinder radius="${base_width/3}" length="${6*itom}" />
-        <origin xyz="0 0 ${3*itom}" />
+        <cylinder radius="${turntable_radius}" length="${turntable_height}" />
       </geometry>
+      <origin xyz="0 0 ${turntable_height/2}" />
     </collision>
-    <inertial>
-      <mass value="50"/> <!-- TODO: Update with proper mass, possibly calculated from Solidworks? -->
-      <inertia ixx="100.0" ixy="0.0" ixz="0.0" iyy="100.0" iyz="0.0" izz="100.0"/> <!-- TODO: Update with proper inertial values, possibly calculated from Solidworks? -->
-    </inertial>
   </link>
   <joint name="turntable_joint" type="continuous">
@@ -25,6 +21,5 @@
     <origin xyz="${base_length/2-base_width/3-3*itom} 0 ${base_height/2}" />
     <axis xyz="0 0 1" />
-    <limit effort="10000.0"  velocity="0.25"/>
-    <dynamics damping="0.7"/>
+    <limit effort="1.0" velocity="1.0"/>
   </joint>
   <transmission name="turntable_tran">
@@ -39,22 +34,17 @@
     </actuator>
   </transmission>
-  <!-- /fold -->
   <link name="lower_arm">
     <visual>
       <geometry>
-        <box size="${4*itom} ${4*itom} ${36*itom}" />
+        <box size="${lower_arm_height} ${lower_arm_width} ${lower_arm_length}" />
       </geometry>
-      <origin xyz="0 0 ${18*itom}" />
+      <origin xyz="${-lower_arm_height/2} 0 ${lower_arm_length/2}" />
     </visual>
     <collision>
       <geometry>
-        <box size="${4*itom} ${4*itom} ${36*itom}" />
+        <box size="${lower_arm_height} ${lower_arm_width} ${lower_arm_length}" />
       </geometry>
-      <origin xyz="0 0 ${18*itom}" />
+      <origin xyz="${-lower_arm_height/2} 0 ${lower_arm_length/2}" />
     </collision>
-    <inertial>
-      <mass value="50"/> <!-- TODO: Update with proper mass, possibly calculated from Solidworks? -->
-      <inertia ixx="100.0" ixy="0.0" ixz="0.0" iyy="100.0" iyz="0.0" izz="100.0"/> <!-- TODO: Update with proper inertial values, possibly calculated from Solidworks? -->
-    </inertial>
   </link>
   <joint name="lower_arm_joint" type="revolute">
@@ -62,7 +52,6 @@
     <child link="lower_arm" />
     <axis xyz="0 1 0" />
-    <origin xyz="0 0 ${6*itom}" />
-    <limit effort="10000.0"  velocity="0.25" lower="${-pi/6}" upper="${3*pi/8}"/>
-    <dynamics damping="5.0"/>
+    <origin xyz="${turntable_radius} 0 ${turntable_height}" />
+    <limit effort="1.0" velocity="1.0" lower="${lower_arm_min}" upper="${lower_arm_max}"/>
   </joint>
   <transmission name="lower_arm_tran">
@@ -80,18 +69,14 @@
     <visual>
       <geometry>
-        <box size="${4*itom} ${4*itom} ${36*itom}" />
+        <box size="${upper_arm_height} ${upper_arm_width} ${upper_arm_length}" />
       </geometry>
-      <origin xyz="0 0 ${18*itom}" />
+      <origin xyz="${-upper_arm_height/2} 0 ${upper_arm_length/2}" />
     </visual>
     <collision>
       <geometry>
-        <box size="${4*itom} ${4*itom} ${36*itom}" />
+        <box size="${upper_arm_height} ${upper_arm_width} ${upper_arm_length}" />
       </geometry>
-      <origin xyz="0 0 ${18*itom}" />
+      <origin xyz="${-upper_arm_height/2} 0 ${upper_arm_length/2}" />
     </collision>
-    <inertial>
-      <mass value="50"/> <!-- TODO: Update with proper mass, possibly calculated from Solidworks? -->
-      <inertia ixx="100.0" ixy="0.0" ixz="0.0" iyy="100.0" iyz="0.0" izz="100.0"/> <!-- TODO: Update with proper inertial values, possibly calculated from Solidworks? -->
-    </inertial>
   </link>
   <joint name="upper_arm_joint" type="revolute">
@@ -99,7 +84,6 @@
     <child link="upper_arm" />
     <axis xyz="0 1 0" />
-    <origin xyz="0 0 ${36*itom}" />
-    <limit effort="10000.0"  velocity="0.25" lower="0.0" upper="${3*pi/8}"/>
-    <dynamics damping="5.0"/>
+    <origin xyz="0 0 ${lower_arm_length}" />
+    <limit effort="1.0" velocity="1.0" lower="${upper_arm_min}" upper="${upper_arm_max}"/>
   </joint>
   <transmission name="upper_arm_tran">
@@ -117,20 +101,21 @@
     <visual>
       <geometry>
-        <box size="${12*itom} ${12*itom} ${4*itom}" />
+        <box size="${scoop_diameter} ${scoop_width} ${scoop_diameter/2}" />
       </geometry>
-      <origin xyz="${6*itom} 0 0" />
+      <origin xyz="${scoop_diameter/2} 0 ${scoop_diameter/4}" />
     </visual>
-    <inertial>
-      <mass value="50"/> <!-- TODO: Update with proper mass, possibly calculated from Solidworks? -->
-      <inertia ixx="100.0" ixy="0.0" ixz="0.0" iyy="100.0" iyz="0.0" izz="100.0"/> <!-- TODO: Update with proper inertial values, possibly calculated from Solidworks? -->
-    </inertial>
+    <collision>
+      <geometry>
+        <box size="${scoop_diameter} ${scoop_width} ${scoop_diameter/2}" />
+      </geometry>
+      <origin xyz="${scoop_diameter/2} 0 ${scoop_diameter/4}" />
+    </collision>
   </link>
   <joint name="scoop_joint" type="revolute">
     <parent link="upper_arm" />
     <child link="scoop" />
-    <origin xyz="0 0 ${36*itom}" />
+    <origin xyz="0 0 ${upper_arm_length}" />
     <axis xyz="0 1 0" />
-    <limit effort="10000.0" velocity="0.25" lower="${-3*pi/8}" upper="${pi/4}" />
-    <dynamics damping="5.0"/>
+    <limit effort="1.0" velocity="1.0" lower="${scoop_min}" upper="${scoop_max}" />
   </joint>
   <transmission name="scoop_tran">

File: src/tfr_description/xacro/model_base.xacro (robot description, xacro)
@@ -17,17 +17,11 @@
         <origin rpy="${pi/2} 0 0" />
       </collision>
-      <inertial>
-        <origin xyz="0 ${wheel_width/2} 0" rpy="0 0 0"/>
-        <mass value="${wheel_mass}"/>
-        <inertia ixx="${(wheel_mass*wheel_radius**2)/2}" ixy="0.0" ixz="0.0" iyy="${(wheel_mass*wheel_width**2)/12}" iyz="0.0" izz="${(wheel_mass*wheel_radius**2)/2}"/>
-      </inertial>
     </link>
     <joint name="${name}_joint" type="continuous">
       <parent link="base_link"/>
       <child link="${name}"/>
-      <origin xyz="${fb*base_length/2 - 16*fb*itom} ${lr*base_width/2 + lr*wheel_width/2} ${-base_height/2}"/>
+      <origin xyz="${fb*base_length/2 - fb*wheel_radius} ${lr*base_width/2 + lr*wheel_width/2} ${-base_height/2}"/>
       <axis xyz="0 1 0"/>
-      <limit effort="100.0"  velocity="100.0"/>
-      <dynamics damping="0.7"/>
+      <limit effort="1.0"  velocity="1.0"/>
     </joint>
   </xacro:macro>
@@ -46,13 +40,11 @@
   </xacro:macro>
   <!--stamp out the "treads" (just individual wheels) -->
-  <xacro:wheel name="left_tread" fb="0" lr="1" />
+  <xacro:wheel name="left_tread" fb="-1" lr="1" />
   <xacro:wheel_tran name="left_tread" />
-  <xacro:wheel name="right_tread" fb = "0" lr="-1" />
+  <xacro:wheel name="right_tread" fb = "-1" lr="-1" />
   <xacro:wheel_tran name="right_tread" />
   <!-- add extra, free-spinning wheels so the robot doesn't wobble in simulation -->
   <xacro:wheel name="left_tread_f" fb="1" lr="1" />
-  <xacro:wheel name="left_tread_b" fb="-1" lr="1" />
   <xacro:wheel name="right_tread_f" fb="1" lr="-1" />
-  <xacro:wheel name="right_tread_b" fb="-1" lr="-1" />
   <!--CHASSIS-->
   <link name="base_link" >
@@ -67,8 +59,4 @@
       </geometry>
     </collision>
-    <inertial>
-      <mass value="${base_mass}"/>
-      <inertia ixx="${base_mass/12*(base_width**2+base_length**2)}" ixy="0.0" ixz="0.0" iyy="${base_mass/12*(base_length**2+base_height**2)}" iyz="0.0" izz="${base_mass/12*(base_width**2+base_height**2)}"/>
-    </inertial>
   </link>
   <!--BIN-->
@@ -76,19 +64,14 @@
     <visual>
       <geometry>
-        <box size="${base_length/3} ${base_width*5/6} ${12*itom}" />
+        <box size="${bin_length} ${bin_width} ${bin_height}" />
       </geometry>
-      <origin xyz="${base_length/6} 0 ${6*itom}" />
+      <origin xyz="${bin_length/2} 0 ${bin_height/2}" />
     </visual>
     <collision>
       <geometry>
-        <box size="${base_length/3} ${base_width*5/6} ${12*itom}" />
+        <box size="${bin_length} ${bin_width} ${bin_height}" />
       </geometry>
-      <origin xyz="${base_length/6} 0 ${6*itom}" />
+      <origin xyz="${bin_length/2} 0 ${bin_height/2}" />
     </collision>
-    <!--TODO: has to be updated with proper values!-->
-    <inertial>
-      <mass value="${base_mass}"/>
-      <inertia ixx="${base_mass/12*(base_width**2+base_length**2)}" ixy="0.0" ixz="0.0" iyy="${base_mass/12*(base_length**2+base_height**2)}" iyz="0.0" izz="${base_mass/12*(base_width**2+base_height**2)}"/>
-    </inertial>
   </link>
   <joint name="bin_joint" type="revolute">
@@ -97,6 +80,5 @@
     <axis xyz="0 -1 0" />
     <origin xyz="${-base_length/2} 0 ${base_height/2}" />
-    <limit effort="10000.0"  velocity="0.25" lower="0" upper="${pi/4}"/>
-    <dynamics damping="5.0"/>
+    <limit effort="1.0"  velocity="1.0" lower="0" upper="${pi/4}"/>
   </joint>
 </robot>

File: src/tfr_description/xacro/model_constants.xacro (robot description, xacro)
@@ -2,13 +2,39 @@
 <robot name="excavator" xmlns:xacro="http://www.ros.org/wiki/xacro">
   <!--shared model level constants-->
+  <xacro:property name="itom" value="0.0254"/> <!-- Inches to meters conversion -->
+  <xacro:property name="dtor" value="${pi/180}"/> <!-- Degrees to radians conversion -->
   <!--drivebase parameters-->
-  <xacro:property name="itom" value="0.0254" /> <!-- Inches to meters conversion -->
-  <xacro:property name="base_width" value="${29*itom}"/>
-  <xacro:property name="base_length" value="${58*itom}"/>
-  <xacro:property name="base_height" value="${2*itom}"/>
-  <xacro:property name="base_mass"   value="5"/>
+  <xacro:property name="base_width" value="${20*itom}"/>
+  <xacro:property name="base_length" value="${50*itom}"/>
+  <xacro:property name="base_height" value="${6*itom}"/>
   <!--wheel parameters-->
-  <xacro:property name="wheel_radius" value="${6*itom}"/>
-  <xacro:property name="wheel_width" value="${6*itom}"/>
-  <xacro:property name="wheel_mass" value="0.5"/>
+  <xacro:property name="wheel_radius" value="${5.5*itom}"/>
+  <xacro:property name="wheel_width" value="${5.75*itom}"/>
+  <!--bin parameters-->
+  <!-- Length of top of bin, length of bottom is 13.86 -->
+  <!-- Using the bigger size as a box instead of making a complex angled shape -->
+  <xacro:property name="bin_length" value="${25.78*itom}"/>
+  <xacro:property name="bin_width" value="${base_width}"/>
+  <xacro:property name="bin_height" value="${12*itom}"/>
+  <!--turntable parameters-->
+  <xacro:property name="turntable_radius" value="${6*itom}"/>
+  <!-- 1" in model plus undefined height for mounting plates and extra components -->
+  <xacro:property name="turntable_height" value="${2*itom}"/>
+  <!--lower arm parameters-->
+  <xacro:property name="lower_arm_length" value="${22*itom}"/>
+  <xacro:property name="lower_arm_width" value="${4*itom}"/>
+  <xacro:property name="lower_arm_height" value="${3.5*itom}"/>
+  <xacro:property name="lower_arm_min" value="${11.74*dtor}"/>
+  <xacro:property name="lower_arm_max" value="${97*dtor}"/>
+  <!--upper arm parameters-->
+  <xacro:property name="upper_arm_length" value="${20*itom}"/>
+  <xacro:property name="upper_arm_width" value="${3.61*itom}"/>
+  <xacro:property name="upper_arm_height" value="${2.5*itom}"/>
+  <xacro:property name="upper_arm_min" value="${0*dtor}"/>
+  <xacro:property name="upper_arm_max" value="${107*dtor}"/>
+  <!--scoop parameters-->
+  <xacro:property name="scoop_width" value="${10*itom}"/>
+  <xacro:property name="scoop_diameter" value="${10.75*itom}"/>
+  <xacro:property name="scoop_min" value="${-50*dtor}"/>
+  <xacro:property name="scoop_max" value="${65*dtor}"/>
 </robot>

Commit message: Tons of edits as per review with Ryan
Made files adhere to the 80 character limit, added file headers.
Also made various tweaks to bits of code: moved Controller to a local
(not global) variable, added an enum for actuators, and removed tons of
build file comments. Also fixed a build issue after rebasing onto master

File: src/tfr_description/xacro/model_arm.xacro (robot description, xacro)
@@ -26,8 +26,10 @@
     <type>transmission_interface/SimpleTransmission</type>
     <joint name="turn_to_base">
-      <hardwareInterface>hardware_interface/EffortJointInterface</hardwareInterface>
+      <hardwareInterface>hardware_interface/EffortJointInterface
+      </hardwareInterface>
     </joint>
     <actuator name="turntable_motor">
-      <hardwareInterface>hardware_interface/EffortJointInterface</hardwareInterface>
+      <hardwareInterface>hardware_interface/EffortJointInterface
+      </hardwareInterface>
       <mechanicalReduction>1</mechanicalReduction>
       <motorTorqueConstant>1</motorTorqueConstant>
@@ -37,5 +39,5 @@
     <visual>
       <geometry>
-        <box size="${lower_arm_height} ${lower_arm_width} ${lower_arm_length}" />
+        <box size="${lower_arm_height} ${lower_arm_width} ${lower_arm_length}"/>
       </geometry>
       <origin xyz="${-lower_arm_height/2} 0 ${lower_arm_length/2}" />
@@ -43,5 +45,5 @@
     <collision>
       <geometry>
-        <box size="${lower_arm_height} ${lower_arm_width} ${lower_arm_length}" />
+        <box size="${lower_arm_height} ${lower_arm_width} ${lower_arm_length}"/>
       </geometry>
       <origin xyz="${-lower_arm_height/2} 0 ${lower_arm_length/2}" />
@@ -53,13 +55,16 @@
     <axis xyz="0 1 0" />
     <origin xyz="${turntable_radius} 0 ${turntable_height}" />
-    <limit effort="1.0" velocity="1.0" lower="${lower_arm_min}" upper="${lower_arm_max}" />
+    <limit effort="1.0" velocity="1.0" lower="${lower_arm_min}"
+          upper="${lower_arm_max}" />
   </joint>
   <transmission name="lower_arm_tran">
     <type>transmission_interface/SimpleTransmission</type>
     <joint name="lower_to_turn">
-      <hardwareInterface>hardware_interface/EffortJointInterface</hardwareInterface>
+      <hardwareInterface>hardware_interface/EffortJointInterface
+      </hardwareInterface>
     </joint>
     <actuator name="lower_motor">
-      <hardwareInterface>hardware_interface/EffortJointInterface</hardwareInterface>
+      <hardwareInterface>hardware_interface/EffortJointInterface
+      </hardwareInterface>
       <mechanicalReduction>1</mechanicalReduction>
       <motorTorqueConstant>1</motorTorqueConstant>
@@ -69,5 +74,5 @@
     <visual>
       <geometry>
-        <box size="${upper_arm_height} ${upper_arm_width} ${upper_arm_length}" />
+        <box size="${upper_arm_height} ${upper_arm_width} ${upper_arm_length}"/>
       </geometry>
       <origin xyz="${-upper_arm_height/2} 0 ${upper_arm_length/2}" />
@@ -75,5 +80,5 @@
     <collision>
       <geometry>
-        <box size="${upper_arm_height} ${upper_arm_width} ${upper_arm_length}" />
+        <box size="${upper_arm_height} ${upper_arm_width} ${upper_arm_length}"/>
       </geometry>
       <origin xyz="${-upper_arm_height/2} 0 ${upper_arm_length/2}" />
@@ -85,13 +90,16 @@
     <axis xyz="0 1 0" />
     <origin xyz="0 0 ${lower_arm_length}" />
-    <limit effort="1.0" velocity="1.0" lower="${upper_arm_min}" upper="${upper_arm_max}" />
+    <limit effort="1.0" velocity="1.0" lower="${upper_arm_min}"
+          upper="${upper_arm_max}" />
   </joint>
   <transmission name="upper_arm_tran">
     <type>transmission_interface/SimpleTransmission</type>
     <joint name="upper_to_lower">
-      <hardwareInterface>hardware_interface/EffortJointInterface</hardwareInterface>
+      <hardwareInterface>hardware_interface/EffortJointInterface
+      </hardwareInterface>
     </joint>
     <actuator name="upper_motor">
-      <hardwareInterface>hardware_interface/EffortJointInterface</hardwareInterface>
+      <hardwareInterface>hardware_interface/EffortJointInterface
+      </hardwareInterface>
       <mechanicalReduction>1</mechanicalReduction>
       <motorTorqueConstant>1</motorTorqueConstant>
@@ -117,13 +125,16 @@
     <origin xyz="0 0 ${upper_arm_length}" />
     <axis xyz="0 1 0" />
-    <limit effort="1.0" velocity="1.0" lower="${scoop_min}" upper="${scoop_max}" />
+    <limit effort="1.0" velocity="1.0" lower="${scoop_min}"
+          upper="${scoop_max}" />
   </joint>
   <transmission name="scoop_tran">
     <type>transmission_interface/SimpleTransmission</type>
     <joint name="end_to_arm">
-      <hardwareInterface>hardware_interface/EffortJointInterface</hardwareInterface>
+      <hardwareInterface>hardware_interface/EffortJointInterface
+      </hardwareInterface>
     </joint>
     <actuator name="end_motor">
-      <hardwareInterface>hardware_interface/EffortJointInterface</hardwareInterface>
+      <hardwareInterface>hardware_interface/EffortJointInterface
+      </hardwareInterface>
       <mechanicalReduction>1</mechanicalReduction>
       <motorTorqueConstant>1</motorTorqueConstant>

File: src/tfr_description/xacro/model_base.xacro (robot description, xacro)
@@ -34,5 +34,6 @@
       <parent link="base_link" />
       <child link="${name}" />
-      <origin xyz="${fb*base_length/2 - fb*wheel_radius} ${lr*base_width/2 + lr*wheel_width/2} ${-base_height/2}" />
+      <origin xyz="${fb*base_length/2 - fb*wheel_radius}
+                  ${lr*base_width/2 + lr*wheel_width/2} ${-base_height/2}" />
       <axis xyz="0 1 0"/>
       <limit effort="1.0" velocity="1.0" />
@@ -44,8 +45,10 @@
       <type>transmission_interface/SimpleTransmission</type>
       <joint name="${name}_joint">
-        <hardwareInterface>hardware_interface/EffortJointInterface</hardwareInterface>
+        <hardwareInterface>hardware_interface/EffortJointInterface
+        </hardwareInterface>
       </joint>
       <actuator name="${name}_motor">
-        <hardwareInterface>hardware_interface/EffortJointInterface</hardwareInterface>
+        <hardwareInterface>hardware_interface/EffortJointInterface
+        </hardwareInterface>
         <mechanicalReduction>1</mechanicalReduction>
         <motorTorqueConstant>1</motorTorqueConstant>

File: src/tfr_description/xacro/model_constants.xacro (robot description, xacro)
@@ -2,6 +2,8 @@
 <robot name="excavator" xmlns:xacro="http://www.ros.org/wiki/xacro">
   <!-- Shared model level constants -->
-  <xacro:property name="itom" value="0.0254" /> <!-- Inches to meters conversion -->
-  <xacro:property name="dtor" value="${pi/180}" /> <!-- Degrees to radians conversion -->
+  <!-- Inches to meters conversion -->
+  <xacro:property name="itom" value="0.0254" />
+  <!-- Degrees to radians conversion -->
+  <xacro:property name="dtor" value="${pi/180}" />
   <!-- Drivebase parameters -->
   <xacro:property name="base_width" value="${20*itom}" />
@@ -13,5 +15,5 @@
   <!-- Bin parameters -->
   <!-- Length of top of bin, length of bottom is 13.86 -->
-  <!-- Using the bigger size as a box instead of making a complex angled shape -->
+  <!-- Using the bigger size as a box instead of making complex angled shape -->
   <xacro:property name="bin_length" value="${25.78*itom}" />
   <xacro:property name="bin_width" value="${base_width}" />
@@ -19,5 +21,5 @@
   <!-- Turntable parameters -->
   <xacro:property name="turntable_radius" value="${6*itom}" />
-  <!-- 1" in model plus undefined height for mounting plates and extra components -->
+  <!-- 1" in model plus undefined height for mounting and extra components -->
   <!-- Rounded to 2" for now -->
   <xacro:property name="turntable_height" value="${2*itom}" />
