Commit message: Updated the bin model
Note: there is a slight tiny gap at the bottom: this is so small it
really isn't relevant for MoveIt.

File: src/tfr_description/xacro/model_arm.xacro (robot description, xacro)
@@ -19,5 +19,5 @@
     <parent link="base_link" />
     <child link="turntable" />
-    <origin xyz="${base_length/2-base_width/3-3*itom} 0 ${base_height/2}" />
+    <origin xyz="${base_length/2-drivebase_beam_width/3-3*itom} 0 ${drivebase_total_height/2}" />
     <axis xyz="0 0 1" />
     <limit effort="1.0" velocity="1.0" />

File: src/tfr_description/xacro/model_base.xacro (robot description, xacro)
@@ -148,24 +148,67 @@
   </joint>
   <!-- BIN -->
-  <link name="bin" >
-    <visual>
-      <geometry>
-        <box size="${bin_length} ${bin_width} ${bin_height}" />
-      </geometry>
-      <origin xyz="${bin_length/2} 0 ${bin_height/2}" />
-    </visual>
-    <collision>
-      <geometry>
-        <box size="${bin_length} ${bin_width} ${bin_height}" />
-      </geometry>
-      <origin xyz="${bin_length/2} 0 ${bin_height/2}" />
-    </collision>
-  </link>
-  <joint name="bin_joint" type="revolute">
+  <link name="bin_back" >
+    <visual>
+      <geometry>
+        <box size="${0.125*itom} ${bin_width} ${bin_height}" />
+      </geometry>
+      <origin xyz="${bin_length} 0 ${-bin_height/2 + bin_height - (9.88 * itom) + (0.5*itom)}" />
+    </visual>
+  </link>
+  <joint name="bin_back_joint" type="revolute">
     <parent link="base_link" />
-    <child link="bin" />
+    <child link="bin_back" />
     <axis xyz="0 -1 0" />
-    <origin xyz="${-base_length/2} 0 ${base_height/2}" />
+    <origin xyz="${-base_length/2} 0 ${drivebase_total_height/2 + (9.88 * itom)}" />
     <limit effort="1.0" velocity="1.0" lower="0" upper="${pi/4}" />
   </joint>
+  <link name="bin_right" >
+    <visual>
+      <geometry>
+        <box size="${bin_length} ${0.125*itom} ${bin_height}"/>
+      </geometry>
+    </visual>
+  </link>
+  <joint name="bin_right_joint" type="fixed">
+    <parent link="bin_back" />
+    <child link="bin_right" />
+    <origin xyz="${bin_length/2} ${-bin_width/2} ${bin_height/2 - (9.88 * itom) + (0.5*itom)}" />
+  </joint>
+  <link name="bin_left" >
+    <visual>
+      <geometry>
+        <box size="${bin_length} ${0.125*itom} ${bin_height}"/>
+      </geometry>
+    </visual>
+  </link>
+  <joint name="bin_left_joint" type="fixed">
+    <parent link="bin_back" />
+    <child link="bin_left" />
+    <origin xyz="${bin_length/2} ${bin_width/2} ${bin_height/2 - (9.88 * itom) + (0.5*itom)}" />
+  </joint>
+  <link name="bin_bottom" >
+    <visual>
+      <geometry>
+        <box size="${13.84*itom} ${bin_width} ${0.125*itom}"/>
+      </geometry>
+    </visual>
+  </link>
+  <joint name="bin_bottom_joint" type="fixed">
+    <parent link="bin_back" />
+    <child link="bin_bottom" />
+    <origin xyz="${(13.84/2)*itom + (bin_length/2) - (sqrt2*itom)} 0 ${-(9.88 * itom) + (0.5 * itom)}" />
+  </joint>
+  <link name="bin_slope" >
+    <visual>
+      <geometry>
+        <box size="${0.125*itom} ${bin_width} ${bin_height*sqrt2}" />
+      </geometry>
+      <origin xyz="0 0 ${-bin_height*sqrt2*0.5}"/>
+    </visual>
+  </link>
+  <joint name="bin_slope_joint" type="fixed">
+    <parent link="bin_back" />
+    <child link="bin_slope" />
+    <origin xyz="0 0 ${(12-9.88) * itom}" rpy="0 ${-pi/4} 0"/>
+  </joint>
 </robot>

File: src/tfr_description/xacro/model_constants.xacro (robot description, xacro)
@@ -7,8 +7,7 @@
   <!-- Degrees to radians conversion -->
   <xacro:property name="dtor" value="${pi/180}" />
+  <xacro:property name="sqrt2" value="1.41421" />
   <!-- Drivebase parameters -->
-  <xacro:property name="base_width" value="${20*itom}" />
   <xacro:property name="base_length" value="${50*itom}" />
-  <xacro:property name="base_height" value="${6*itom}" />
   <xacro:property name="tube_width" value="${2*itom}" />
   <xacro:property name="drivebase_beam_width" value="${11.5*itom}" />
@@ -29,6 +28,6 @@
   <!-- Using the bigger size as a box instead of making complex angled shape -->
   <xacro:property name="bin_length" value="${25.78*itom}" />
-  <xacro:property name="bin_width" value="${base_width}" />
-  <xacro:property name="bin_height" value="${12*itom}" />
+  <xacro:property name="bin_width" value="${11*itom}" />
+  <xacro:property name="bin_height" value="${11.5*itom}" />
   <!-- Turntable parameters -->
   <xacro:property name="turntable_radius" value="${6*itom}" />

Commit message: Fixed missing tread flap and shifted arm
Shifted the arm on the turntable to its proper position
(may want to verify this again once it's assembled to ensure that
the CAD model is right)

File: src/tfr_description/xacro/model_arm.xacro (robot description, xacro)
@@ -19,5 +19,5 @@
     <parent link="base_link" />
     <child link="turntable" />
-    <origin xyz="${base_length/2-drivebase_beam_width/3-3*itom} 0 ${drivebase_total_height/2}" />
+    <origin xyz="${base_length/2-turntable_radius} 0 ${drivebase_front_beam_height/2}" />
     <axis xyz="0 0 1" />
     <limit effort="1.0" velocity="1.0" />
@@ -54,5 +54,5 @@
     <child link="lower_arm" />
     <axis xyz="0 1 0" />
-    <origin xyz="${turntable_radius} 0 ${turntable_height}" />
+    <origin xyz="${-2.165*itom} 0 ${turntable_height}" />
     <limit effort="1.0" velocity="1.0" lower="${lower_arm_min}"
           upper="${lower_arm_max}" />

File: src/tfr_description/xacro/model_base.xacro (robot description, xacro)
@@ -145,4 +145,17 @@
     <parent link="tread_right_link" />
     <child link="front_right_slope_link" />
+    <origin xyz="${tread_mid_length/2} 0.0 ${tread_mid_height/2}" rpy="0.0 ${(180-164.1)*dtor} 0.0" />
+  </joint>
+  <link name="front_left_slope_link">
+    <visual>
+      <geometry>
+        <box size="${tread_slope_length} ${tread_width} ${1.25*itom}"/>
+      </geometry>
+      <origin xyz="${tread_slope_length/2} 0.0 ${-1.25/2*itom}" />
+    </visual>
+  </link>
+  <joint name="front_left_slope_joint" type="fixed">
+    <parent link="tread_left_link" />
+    <child link="front_left_slope_link" />
     <origin xyz="${tread_mid_length/2} 0.0 ${tread_mid_height/2}" rpy="0.0 ${(180-164.1)*dtor} 0.0" />
   </joint>

File: src/tfr_description/xacro/model_constants.xacro (robot description, xacro)
@@ -31,8 +31,8 @@
   <xacro:property name="bin_height" value="${11.5*itom}" />
   <!-- Turntable parameters -->
-  <xacro:property name="turntable_radius" value="${6*itom}" />
+  <xacro:property name="turntable_radius" value="${4.92*itom}" />
   <!-- 1" in model plus undefined height for mounting and extra components -->
   <!-- Rounded to 2" for now -->
-  <xacro:property name="turntable_height" value="${2*itom}" />
+  <xacro:property name="turntable_height" value="${1.2*itom}" />
   <!-- Lower arm parameters -->
   <xacro:property name="lower_arm_length" value="${22*itom}" />

Commit message: Updated the arm dimensions based on real measurements.
Next step is to re-add the collision tags I removed.

File: src/tfr_description/xacro/model_arm.xacro (robot description, xacro)
@@ -39,14 +39,8 @@
     <visual>
       <geometry>
-        <box size="${lower_arm_height} ${lower_arm_width} ${lower_arm_length}"/>
+        <box size="${lower_arm_height} ${lower_arm_width} ${lower_arm_primary_length}"/>
       </geometry>
-      <origin xyz="${-lower_arm_height/2} 0 ${lower_arm_length/2}" />
+      <origin xyz="${-lower_arm_height/2} 0 ${14*itom}" />
     </visual>
-    <collision>
-      <geometry>
-        <box size="${lower_arm_height} ${lower_arm_width} ${lower_arm_length}"/>
-      </geometry>
-      <origin xyz="${-lower_arm_height/2} 0 ${lower_arm_length/2}" />
-    </collision>
   </link>
   <joint name="lower_arm_joint" type="revolute">
@@ -71,4 +65,29 @@
     </actuator>
   </transmission>
+  <link name="lower_arm_bottom">
+    <visual>
+      <geometry>
+        <box size="${0.25*itom} ${lower_arm_width} ${lower_arm_length - lower_arm_primary_length}"/>
+      </geometry>
+    </visual>
+  </link>
+  <joint name="lower_arm_bottom_joint" type="fixed">
+    <parent link="lower_arm" />
+    <child link="lower_arm_bottom" />
+    <origin xyz="${-0.125*itom} 0 ${(lower_arm_length - lower_arm_primary_length)/2}" />
+  </joint>
+  <link name="lower_arm_slope">
+    <visual>
+      <geometry>
+        <box size="${0.25*itom} ${lower_arm_width} ${(lower_arm_length - lower_arm_primary_length) * sqrt2}"/>
+      </geometry>
+      <origin xyz="${0.125*itom} 0 ${-(lower_arm_length - lower_arm_primary_length) / 2 * sqrt2}" rpy="0 0 0" />
+    </visual>
+  </link>
+  <joint name="lower_arm_slope_joint" type="fixed">
+    <parent link="lower_arm" />
+    <child link="lower_arm_slope" />
+    <origin xyz="${-lower_arm_height} 0 ${(lower_arm_length - lower_arm_primary_length)}" rpy="0 ${-44*dtor} 0"/>
+  </joint>
   <link name="upper_arm">
     <visual>
@@ -123,5 +142,5 @@
     <parent link="upper_arm" />
     <child link="scoop" />
-    <origin xyz="0 0 ${upper_arm_length}" />
+    <origin xyz="${1.5*itom} 0 ${upper_arm_length - (0.875*itom)}" />
     <axis xyz="0 1 0" />
     <limit effort="1.0" velocity="1.0" lower="${scoop_min}"

File: src/tfr_description/xacro/model_constants.xacro (robot description, xacro)
@@ -35,17 +35,18 @@
   <!-- Lower arm parameters -->
   <xacro:property name="lower_arm_length" value="${22*itom}" />
+  <xacro:property name="lower_arm_primary_length" value="${16*itom}" />
   <xacro:property name="lower_arm_width" value="${4*itom}" />
-  <xacro:property name="lower_arm_height" value="${3.5*itom}" />
+  <xacro:property name="lower_arm_height" value="${6*itom}" />
   <xacro:property name="lower_arm_min" value="${11.74*dtor}" />
   <xacro:property name="lower_arm_max" value="${97*dtor}" />
   <!-- Upper arm parameters -->
   <xacro:property name="upper_arm_length" value="${20*itom}" />
-  <xacro:property name="upper_arm_width" value="${3.61*itom}" />
-  <xacro:property name="upper_arm_height" value="${2.5*itom}" />
+  <xacro:property name="upper_arm_width" value="${3.625*itom}" />
+  <xacro:property name="upper_arm_height" value="${5*itom}" />
   <xacro:property name="upper_arm_min" value="${0*dtor}" />
   <xacro:property name="upper_arm_max" value="${107*dtor}" />
   <!-- Scoop parameters -->
   <xacro:property name="scoop_width" value="${10*itom}" />
-  <xacro:property name="scoop_diameter" value="${10.75*itom}" />
+  <xacro:property name="scoop_diameter" value="${10.5*itom}" />
   <xacro:property name="scoop_min" value="${-50*dtor}" />
   <xacro:property name="scoop_max" value="${65*dtor}" />

Commit message: Updated the arm angles
Please note that the lower arm lower limit is temporarily and
arbitrarily set to "a bit higher than the turntable" so that
it doesn't clip. This should be updated with empirical data
once the arm is mounted.

File: src/tfr_description/xacro/model_arm.xacro (robot description, xacro)
@@ -125,5 +125,5 @@
     </actuator>
   </transmission>
-  <link name="scoop" >
+  <link name="scoop">
     <visual>
       <geometry>

File: src/tfr_description/xacro/model_constants.xacro (robot description, xacro)
@@ -38,16 +38,16 @@
   <xacro:property name="lower_arm_width" value="${4*itom}" />
   <xacro:property name="lower_arm_height" value="${6*itom}" />
-  <xacro:property name="lower_arm_min" value="${11.74*dtor}" />
-  <xacro:property name="lower_arm_max" value="${97*dtor}" />
+  <xacro:property name="lower_arm_min" value="${5.5*dtor}" />
+  <xacro:property name="lower_arm_max" value="${85*dtor}" /> <!-- TODO: must be determined once mounted-->
   <!-- Upper arm parameters -->
   <xacro:property name="upper_arm_length" value="${20*itom}" />
   <xacro:property name="upper_arm_width" value="${3.625*itom}" />
   <xacro:property name="upper_arm_height" value="${5*itom}" />
-  <xacro:property name="upper_arm_min" value="${0*dtor}" />
-  <xacro:property name="upper_arm_max" value="${107*dtor}" />
+  <xacro:property name="upper_arm_min" value="${48*dtor}" />
+  <xacro:property name="upper_arm_max" value="${113*dtor}" />
   <!-- Scoop parameters -->
   <xacro:property name="scoop_width" value="${10*itom}" />
   <xacro:property name="scoop_diameter" value="${10.5*itom}" />
-  <xacro:property name="scoop_min" value="${-50*dtor}" />
-  <xacro:property name="scoop_max" value="${65*dtor}" />
+  <xacro:property name="scoop_min" value="${-61*dtor}" />
+  <xacro:property name="scoop_max" value="${78*dtor}" />
 </robot>

Commit message: Changed the turntable to a revolute joint
This is to prevent the arm from trying to do a full 360, which
has the possibility of ripping wires out.

File: src/tfr_description/xacro/model_arm.xacro (robot description, xacro)
@@ -16,10 +16,10 @@
     </collision>
   </link>
-  <joint name="turntable_joint" type="continuous">
+  <joint name="turntable_joint" type="revolute">
     <parent link="base_link" />
     <child link="turntable" />
     <origin xyz="${base_length/2-turntable_radius} 0 ${drivebase_front_beam_height/2}" />
     <axis xyz="0 0 1" />
-    <limit effort="1.0" velocity="1.0" />
+    <limit effort="1.0" velocity="1.0" lower="${-pi}" upper="${pi}" />
   </joint>
   <transmission name="turntable_tran">

Commit message: Got the new model ready for MoveIt

File: src/tfr_description/xacro/model_arm.xacro (robot description, xacro)
@@ -43,4 +43,10 @@
       <origin xyz="${-lower_arm_height/2} 0 ${14*itom}" />
     </visual>
+    <collision>
+      <geometry>
+        <box size="${lower_arm_height} ${lower_arm_width} ${lower_arm_primary_length}"/>
+      </geometry>
+      <origin xyz="${-lower_arm_height/2} 0 ${14*itom}" />
+    </collision>
   </link>
   <joint name="lower_arm_joint" type="revolute">
@@ -71,4 +77,9 @@
       </geometry>
     </visual>
+    <collision>
+      <geometry>
+        <box size="${0.25*itom} ${lower_arm_width} ${lower_arm_length - lower_arm_primary_length}"/>
+      </geometry>
+    </collision>
   </link>
   <joint name="lower_arm_bottom_joint" type="fixed">
@@ -84,4 +95,10 @@
       <origin xyz="${0.125*itom} 0 ${-(lower_arm_length - lower_arm_primary_length) / 2 * sqrt2}" rpy="0 0 0" />
     </visual>
+    <collision>
+      <geometry>
+        <box size="${0.25*itom} ${lower_arm_width} ${(lower_arm_length - lower_arm_primary_length) * sqrt2}"/>
+      </geometry>
+      <origin xyz="${0.125*itom} 0 ${-(lower_arm_length - lower_arm_primary_length) / 2 * sqrt2}" rpy="0 0 0" />
+    </collision>
   </link>
   <joint name="lower_arm_slope_joint" type="fixed">

File: src/tfr_description/xacro/model_base.xacro (robot description, xacro)
@@ -64,6 +64,11 @@
       </geometry>
     </visual>
-  </link>
-  <joint name="tread_left_joint" type="fixed">
+    <collision>
+      <geometry>
+        <box size="${tread_mid_length} ${tread_width} ${tread_mid_height}"/>
+      </geometry>
+    </collision>
+  </link>
+  <joint name="left_tread_joint" type="fixed">
     <parent link="base_link" />
     <child link="tread_left_link" />
@@ -76,6 +81,11 @@
       </geometry>
     </visual>
-  </link>
-  <joint name="tread_right_joint" type="fixed">
+    <collision>
+      <geometry>
+        <box size="${tread_mid_length} ${tread_width} ${tread_mid_height}"/>
+      </geometry>
+    </collision>
+  </link>
+  <joint name="right_tread_joint" type="fixed">
     <parent link="base_link" />
     <child link="tread_right_link" />
@@ -89,4 +99,10 @@
       <origin rpy="${pi/2} 0.0 0.0" />
     </visual>
+    <collision>
+      <geometry>
+        <cylinder radius="${tread_end_radius}" length="${tread_width}" />
+      </geometry>
+      <origin rpy="${pi/2} 0.0 0.0" />
+    </collision>
   </link>
   <joint name="tread_left_front_joint" type="fixed">
@@ -102,4 +118,10 @@
       <origin rpy="${pi/2} 0.0 0.0" />
     </visual>
+    <collision>
+      <geometry>
+        <cylinder radius="${tread_end_radius}" length="${tread_width}" />
+      </geometry>
+      <origin rpy="${pi/2} 0.0 0.0" />
+    </collision>
   </link>
   <joint name="tread_left_rear_joint" type="fixed">
@@ -115,4 +137,10 @@
       <origin rpy="${pi/2} 0.0 0.0" />
     </visual>
+    <collision>
+      <geometry>
+        <cylinder radius="${tread_end_radius}" length="${tread_width}" />
+      </geometry>
+      <origin rpy="${pi/2} 0.0 0.0" />
+    </collision>
   </link>
   <joint name="tread_right_front_joint" type="fixed">
@@ -128,4 +156,10 @@
       <origin rpy="${pi/2} 0.0 0.0" />
     </visual>
+    <collision>
+      <geometry>
+        <cylinder radius="${tread_end_radius}" length="${tread_width}" />
+      </geometry>
+      <origin rpy="${pi/2} 0.0 0.0" />
+    </collision>
   </link>
   <joint name="tread_right_rear_joint" type="fixed">
@@ -141,4 +175,10 @@
       <origin xyz="${tread_slope_length/2} 0.0 ${-1.25/2*itom}" />
     </visual>
+    <collision>
+      <geometry>
+        <box size="${tread_slope_length} ${tread_width} ${1.25*itom}"/>
+      </geometry>
+      <origin xyz="${tread_slope_length/2} 0.0 ${-1.25/2*itom}" />
+    </collision>
   </link>
   <joint name="front_right_slope_joint" type="fixed">
@@ -154,4 +194,10 @@
       <origin xyz="${tread_slope_length/2} 0.0 ${-1.25/2*itom}" />
     </visual>
+    <collision>
+      <geometry>
+        <box size="${tread_slope_length} ${tread_width} ${1.25*itom}"/>
+      </geometry>
+      <origin xyz="${tread_slope_length/2} 0.0 ${-1.25/2*itom}" />
+    </collision>
   </link>
   <joint name="front_left_slope_joint" type="fixed">
@@ -168,6 +214,12 @@
       <origin xyz="${bin_length} 0 ${-bin_height/2 + bin_height - (9.88 * itom) + (0.5*itom)}" />
     </visual>
-  </link>
-  <joint name="bin_back_joint" type="revolute">
+    <collision>
+      <geometry>
+        <box size="${0.125*itom} ${bin_width} ${bin_height}" />
+      </geometry>
+      <origin xyz="${bin_length} 0 ${-bin_height/2 + bin_height - (9.88 * itom) + (0.5*itom)}" />
+    </collision>
+  </link>
+  <joint name="bin_joint" type="revolute">
     <parent link="base_link" />
     <child link="bin_back" />
@@ -182,4 +234,9 @@
       </geometry>
     </visual>
+    <collision>
+      <geometry>
+        <box size="${bin_length} ${0.125*itom} ${bin_height}"/>
+      </geometry>
+    </collision>
   </link>
   <joint name="bin_right_joint" type="fixed">
@@ -194,4 +251,9 @@
       </geometry>
     </visual>
+    <collision>
+      <geometry>
+        <box size="${bin_length} ${0.125*itom} ${bin_height}"/>
+      </geometry>
+    </collision>
   </link>
   <joint name="bin_left_joint" type="fixed">
@@ -206,4 +268,9 @@
       </geometry>
     </visual>
+    <collision>
+      <geometry>
+        <box size="${13.84*itom} ${bin_width} ${0.125*itom}"/>
+      </geometry>
+    </collision>
   </link>
   <joint name="bin_bottom_joint" type="fixed">
@@ -219,4 +286,10 @@
       <origin xyz="0 0 ${-bin_height*sqrt2*0.5}"/>
     </visual>
+    <collision>
+      <geometry>
+        <box size="${0.125*itom} ${bin_width} ${bin_height*sqrt2}" />
+      </geometry>
+      <origin xyz="0 0 ${-bin_height*sqrt2*0.5}"/>
+    </collision>
   </link>
   <joint name="bin_slope_joint" type="fixed">

Commit message: Added a fix for the arm dumping issue
Turns out that adding a delay between dumping positions fixes
the issue.

File: src/tfr_description/xacro/model_arm.xacro (robot description, xacro)
@@ -21,5 +21,5 @@
     <origin xyz="${base_length/2-turntable_radius} 0 ${drivebase_front_beam_height/2}" />
     <axis xyz="0 0 1" />
-    <limit effort="1.0" velocity="1.0" lower="${-pi}" upper="${pi}" />
+    <limit effort="1.0" velocity="1.0" lower="${-1.1*pi}" upper="${1.1*pi}" />
   </joint>
   <transmission name="turntable_tran">

Commit message: flipped turntable around

File: src/tfr_description/xacro/model_arm.xacro (robot description, xacro)
@@ -7,5 +7,5 @@
         <cylinder radius="${turntable_radius}" length="${turntable_height}" />
       </geometry>
-      <origin xyz="0 0 ${turntable_height/2}" />
+      <origin xyz="0 0 ${turntable_height/2}" rpy="0 0 ${pi}" />
     </visual>
     <collision>
@@ -13,5 +13,5 @@
         <cylinder radius="${turntable_radius}" length="${turntable_height}" />
       </geometry>
-      <origin xyz="0 0 ${turntable_height/2}" />
+      <origin xyz="0 0 ${turntable_height/2}" rpy="0 0 ${pi}" />
     </collision>
   </link>
@@ -19,5 +19,5 @@
     <parent link="base_link" />
     <child link="turntable" />
-    <origin xyz="${base_length/2-turntable_radius} 0 ${drivebase_front_beam_height/2}" />
+    <origin xyz="${base_length/2-turntable_radius} 0 ${drivebase_front_beam_height/2}" rpy="0 0 ${pi}" />
     <axis xyz="0 0 1" />
     <limit effort="1.0" velocity="1.0" lower="${-1.1*pi}" upper="${1.1*pi}" />
