Commit message: Fixed the bin model so that the limits make sense
Fixed the rotation axis of the bin (flipped it) so that now the limits
are actually in order and rotation goes the right way.

File: src/tfr_description/xacro/model_base.xacro (robot description, xacro)
@@ -95,7 +95,7 @@
     <parent link="base_link" />
     <child link="bin" />
-    <axis xyz="0 1 0" />
+    <axis xyz="0 -1 0" />
     <origin xyz="${-base_length/2} 0 ${base_height/2}" />
-    <limit effort="10000.0"  velocity="0.25" lower="0.0" upper="${-pi/4}"/>
+    <limit effort="10000.0"  velocity="0.25" lower="0" upper="${pi/4}"/>
     <dynamics damping="5.0"/>
   </joint>

Commit message: Updated the drivebase model with accurate dimensions

File: src/tfr_description/xacro/model_base.xacro (robot description, xacro)
@@ -5,11 +5,53 @@
     <visual>
       <geometry>
-        <box size="${base_length} ${base_width} ${base_height}" />
+        <box size="${base_length} ${tube_width} ${drivebase_total_height}"/>
       </geometry>
+      <origin xyz="0 ${drivebase_beam_width / 2 + tube_width / 2} 0" />
+    </visual>
+    <visual>
+      <geometry>
+        <box size="${base_length} ${tube_width} ${drivebase_total_height}"/>
+      </geometry>
+      <origin xyz="0 ${-drivebase_beam_width / 2 - tube_width / 2} 0" />
+    </visual>
+    <!-- Front beam -->
+    <visual>
+      <geometry>
+        <box size="${tube_width} ${drivebase_beam_width} ${drivebase_front_beam_height}"/>
+      </geometry>
+      <origin xyz="${base_length / 2 - tube_width / 2} 0 ${drivebase_front_beam_height / 2 - drivebase_total_height / 2}" />
+    </visual>
+    <!-- Rear beam -->
+    <visual>
+      <geometry>
+        <box size="${tube_width} ${drivebase_beam_width} ${drivebase_total_height}"/>
+      </geometry>
+      <origin xyz="${tube_width / 2 - base_length / 2} 0 0" />
     </visual>
     <collision>
       <geometry>
-        <box size="${base_length} ${base_width} ${base_height}" />
+        <box size="${base_length} ${tube_width} ${drivebase_total_height}"/>
       </geometry>
+      <origin xyz="0 ${drivebase_beam_width / 2 + tube_width / 2} 0" />
+    </collision>
+    <collision>
+      <geometry>
+        <box size="${base_length} ${tube_width} ${drivebase_total_height}"/>
+      </geometry>
+      <origin xyz="0 ${-drivebase_beam_width / 2 - tube_width / 2} 0" />
+    </collision>
+    <!-- Front beam -->
+    <collision>
+      <geometry>
+        <box size="${tube_width} ${drivebase_beam_width} ${drivebase_front_beam_height}"/>
+      </geometry>
+      <origin xyz="${base_length / 2 - tube_width / 2} 0 ${drivebase_front_beam_height / 2 - drivebase_total_height / 2}" />
+    </collision>
+    <!-- Rear beam -->
+    <collision>
+      <geometry>
+        <box size="${tube_width} ${drivebase_beam_width} ${drivebase_total_height}"/>
+      </geometry>
+      <origin xyz="${tube_width / 2 - base_length / 2} 0 0" />
     </collision>
   </link>

File: src/tfr_description/xacro/model_constants.xacro (robot description, xacro)
@@ -11,4 +11,8 @@
   <xacro:property name="base_length" value="${50*itom}" />
   <xacro:property name="base_height" value="${6*itom}" />
+  <xacro:property name="tube_width" value="${2*itom}" />
+  <xacro:property name="drivebase_beam_width" value="${11.5*itom}" />
+  <xacro:property name="drivebase_front_beam_height" value="${4*itom}" />
+  <xacro:property name="drivebase_total_height" value="${6*itom}" />
   <!-- Wheel parameters -->
   <xacro:property name="wheel_radius" value="${5.5*itom}" />

Commit message: Updated the model with a simplified tread
Exiting to windows to do more precise measurements, will update
with a proper sloped model next commit.

File: src/tfr_description/xacro/model_base.xacro (robot description, xacro)
@@ -57,53 +57,77 @@
   </link>
   <!-- DRIVEBASE -->
-  <!-- A macro for creating a wheel with a link and joint -->
-  <xacro:macro name="wheel" params="name fb lr">
-    <link name="${name}">
-      <visual>
-        <geometry>
-          <cylinder radius="${wheel_radius}" length="${wheel_width}" />
-        </geometry>
-        <origin rpy="${pi/2} 0 0" />
-      </visual>
-      <collision>
-        <geometry>
-          <cylinder radius="${wheel_radius}" length="${wheel_width}" />
-        </geometry>
-        <origin rpy="${pi/2} 0 0" />
-      </collision>
-    </link>
-    <joint name="${name}_joint" type="continuous">
-      <parent link="base_link" />
-      <child link="${name}" />
-      <origin xyz="${fb*base_length/2 - fb*wheel_radius}
-                  ${lr*base_width/2 + lr*wheel_width/2} ${-base_height/2}" />
-      <axis xyz="0 1 0"/>
-      <limit effort="1.0" velocity="1.0" />
-    </joint>
-  </xacro:macro>
-  <!-- A macro for creating a wheel transmission -->
-  <xacro:macro name="wheel_tran" params="name">
-    <transmission name="${name}_tran">
-      <type>transmission_interface/SimpleTransmission</type>
-      <joint name="${name}_joint">
-        <hardwareInterface>hardware_interface/EffortJointInterface
-        </hardwareInterface>
-      </joint>
-      <actuator name="${name}_motor">
-        <hardwareInterface>hardware_interface/EffortJointInterface
-        </hardwareInterface>
-        <mechanicalReduction>1</mechanicalReduction>
-        <motorTorqueConstant>1</motorTorqueConstant>
-      </actuator>
-    </transmission>
-  </xacro:macro>
-  <!-- Create the "treads" (just individual wheels) -->
-  <xacro:wheel name="left_tread" fb="-1" lr="1" />
-  <xacro:wheel_tran name="left_tread" />
-  <xacro:wheel name="right_tread" fb = "-1" lr="-1" />
-  <xacro:wheel_tran name="right_tread" />
-  <!-- Add extra free-spinning wheels for the other end of the robot -->
-  <xacro:wheel name="left_tread_f" fb="1" lr="1" />
-  <xacro:wheel name="right_tread_f" fb="1" lr="-1" />
+  <!-- A general tread huge block: may be refined later for slightly better operational motion -->
+  <link name="tread_left_link">
+    <visual>
+      <geometry>
+        <box size="${tread_mid_length} ${tread_width} ${tread_mid_height}"/>
+      </geometry>
+    </visual>
+  </link>
+  <joint name="tread_left_joint" type="fixed">
+    <parent link="base_link" />
+    <child link="tread_left_link" />
+    <origin xyz="0 ${(drivebase_beam_width / 2) + tube_width + (tread_width / 2)} 0" />
+  </joint>
+  <link name="tread_right_link">
+    <visual>
+      <geometry>
+        <box size="${tread_mid_length} ${tread_width} ${tread_mid_height}"/>
+      </geometry>
+    </visual>
+  </link>
+  <joint name="tread_right_joint" type="fixed">
+    <parent link="base_link" />
+    <child link="tread_right_link" />
+    <origin xyz="0 ${-(drivebase_beam_width / 2) - tube_width - (tread_width / 2)} 0" />
+  </joint>
+  <link name="tread_left_front_link">
+    <visual>
+      <geometry>
+        <box size="${tread_end_length} ${tread_width} ${tread_end_height}"/>
+      </geometry>
+    </visual>
+  </link>
+  <joint name="tread_left_front_joint" type="fixed">
+    <parent link="tread_left_link" />
+    <child link="tread_left_front_link" />
+    <origin xyz="${(tread_mid_length / 2) + (tread_end_length / 2)} 0 ${(tread_end_height / 2) - (tread_mid_height / 2)}" />
+  </joint>
+  <link name="tread_left_rear_link">
+    <visual>
+      <geometry>
+        <box size="${tread_end_length} ${tread_width} ${tread_end_height}"/>
+      </geometry>
+    </visual>
+  </link>
+  <joint name="tread_left_rear_joint" type="fixed">
+    <parent link="tread_left_link" />
+    <child link="tread_left_rear_link" />
+    <origin xyz="${-(tread_mid_length / 2) - (tread_end_length / 2)} 0 ${(tread_end_height / 2) - (tread_mid_height / 2)}" />
+  </joint>
+  <link name="tread_right_front_link">
+    <visual>
+      <geometry>
+        <box size="${tread_end_length} ${tread_width} ${tread_end_height}"/>
+      </geometry>
+    </visual>
+  </link>
+  <joint name="tread_right_front_joint" type="fixed">
+    <parent link="tread_right_link" />
+    <child link="tread_right_front_link" />
+    <origin xyz="${(tread_mid_length / 2) + (tread_end_length / 2)} 0 ${(tread_end_height / 2) - (tread_mid_height / 2)}" />
+  </joint>
+  <link name="tread_right_rear_link">
+    <visual>
+      <geometry>
+        <box size="${tread_end_length} ${tread_width} ${tread_end_height}"/>
+      </geometry>
+    </visual>
+  </link>
+  <joint name="tread_right_rear_joint" type="fixed">
+    <parent link="tread_right_link" />
+    <child link="tread_right_rear_link" />
+    <origin xyz="${-(tread_mid_length / 2) - (tread_end_length / 2)} 0 ${(tread_end_height / 2) - (tread_mid_height / 2)}" />
+  </joint>
   <!-- BIN -->
   <link name="bin" >

File: src/tfr_description/xacro/model_constants.xacro (robot description, xacro)
@@ -15,4 +15,10 @@
   <xacro:property name="drivebase_front_beam_height" value="${4*itom}" />
   <xacro:property name="drivebase_total_height" value="${6*itom}" />
+  <!-- Drivetrain parameters -->
+  <xacro:property name="tread_end_height" value="${11*itom}" />
+  <xacro:property name="tread_end_length" value="${11*itom}" />
+  <xacro:property name="tread_mid_height" value="${12.89*itom}" />
+  <xacro:property name="tread_mid_length" value="${base_length - (tread_end_length * 2)}" />
+  <xacro:property name="tread_width" value="${5.75*itom}" />
   <!-- Wheel parameters -->
   <xacro:property name="wheel_radius" value="${5.5*itom}" />

Commit message: Updated tread dimensions more
These should probably be remeasured just in case: some things
weren't lining up quite right.

File: src/tfr_description/xacro/model_base.xacro (robot description, xacro)
@@ -68,5 +68,5 @@
     <parent link="base_link" />
     <child link="tread_left_link" />
-    <origin xyz="0 ${(drivebase_beam_width / 2) + tube_width + (tread_width / 2)} 0" />
+    <origin xyz="0 ${tread_spacing / 2 + tread_width / 2} 0" />
   </joint>
   <link name="tread_right_link">
@@ -80,11 +80,12 @@
     <parent link="base_link" />
     <child link="tread_right_link" />
-    <origin xyz="0 ${-(drivebase_beam_width / 2) - tube_width - (tread_width / 2)} 0" />
+    <origin xyz="0 ${-tread_spacing / 2 - tread_width / 2} 0" />
   </joint>
   <link name="tread_left_front_link">
     <visual>
       <geometry>
-        <box size="${tread_end_length} ${tread_width} ${tread_end_height}"/>
+        <cylinder radius="${tread_end_radius}" length="${tread_width}" />
       </geometry>
+      <origin rpy="${pi/2} 0.0 0.0" />
     </visual>
   </link>
@@ -92,11 +93,12 @@
     <parent link="tread_left_link" />
     <child link="tread_left_front_link" />
-    <origin xyz="${(tread_mid_length / 2) + (tread_end_length / 2)} 0 ${(tread_end_height / 2) - (tread_mid_height / 2)}" />
+    <origin xyz="${intertread_length / 2} 0 ${-1.38*itom}" />
   </joint>
   <link name="tread_left_rear_link">
     <visual>
       <geometry>
-        <box size="${tread_end_length} ${tread_width} ${tread_end_height}"/>
+        <cylinder radius="${tread_end_radius}" length="${tread_width}" />
       </geometry>
+      <origin rpy="${pi/2} 0.0 0.0" />
     </visual>
   </link>
@@ -104,11 +106,12 @@
     <parent link="tread_left_link" />
     <child link="tread_left_rear_link" />
-    <origin xyz="${-(tread_mid_length / 2) - (tread_end_length / 2)} 0 ${(tread_end_height / 2) - (tread_mid_height / 2)}" />
+    <origin xyz="${-intertread_length / 2} 0 ${-1.38*itom}" />
   </joint>
   <link name="tread_right_front_link">
     <visual>
       <geometry>
-        <box size="${tread_end_length} ${tread_width} ${tread_end_height}"/>
+        <cylinder radius="${tread_end_radius}" length="${tread_width}" />
       </geometry>
+      <origin rpy="${pi/2} 0.0 0.0" />
     </visual>
   </link>
@@ -116,11 +119,12 @@
     <parent link="tread_right_link" />
     <child link="tread_right_front_link" />
-    <origin xyz="${(tread_mid_length / 2) + (tread_end_length / 2)} 0 ${(tread_end_height / 2) - (tread_mid_height / 2)}" />
+    <origin xyz="${intertread_length / 2} 0 ${-1.38*itom}" />
   </joint>
   <link name="tread_right_rear_link">
     <visual>
       <geometry>
-        <box size="${tread_end_length} ${tread_width} ${tread_end_height}"/>
+        <cylinder radius="${tread_end_radius}" length="${tread_width}" />
       </geometry>
+      <origin rpy="${pi/2} 0.0 0.0" />
     </visual>
   </link>
@@ -128,5 +132,18 @@
     <parent link="tread_right_link" />
     <child link="tread_right_rear_link" />
-    <origin xyz="${-(tread_mid_length / 2) - (tread_end_length / 2)} 0 ${(tread_end_height / 2) - (tread_mid_height / 2)}" />
+    <origin xyz="${-intertread_length / 2} 0 ${-1.38*itom}" />
+  </joint>
+  <link name="front_right_slope_link">
+    <visual>
+      <geometry>
+        <box size="${tread_slope_length} ${tread_width} ${1.25*itom}"/>
+      </geometry>
+      <origin xyz="${tread_slope_length/2} 0.0 ${-1.25/2*itom}" />
+    </visual>
+  </link>
+  <joint name="front_right_slope_joint" type="fixed">
+    <parent link="tread_right_link" />
+    <child link="front_right_slope_link" />
+    <origin xyz="${tread_mid_length/2} 0.0 ${tread_mid_height/2}" rpy="0.0 ${(180-164.1)*dtor} 0.0" />
   </joint>
   <!-- BIN -->

File: src/tfr_description/xacro/model_constants.xacro (robot description, xacro)
@@ -18,10 +18,11 @@
   <xacro:property name="tread_end_height" value="${11*itom}" />
   <xacro:property name="tread_end_length" value="${11*itom}" />
-  <xacro:property name="tread_mid_height" value="${12.89*itom}" />
-  <xacro:property name="tread_mid_length" value="${base_length - (tread_end_length * 2)}" />
+  <xacro:property name="tread_end_radius" value="${(5.5+1.25)*itom}" />
+  <xacro:property name="tread_mid_height" value="${(12.89+(1.25*2))*itom}" />
+  <xacro:property name="tread_mid_length" value="${24*itom}" />
   <xacro:property name="tread_width" value="${5.75*itom}" />
-  <!-- Wheel parameters -->
-  <xacro:property name="wheel_radius" value="${5.5*itom}" />
-  <xacro:property name="wheel_width" value="${5.75*itom}" />
+  <xacro:property name="tread_spacing" value="${16*itom}" />
+  <xacro:property name="intertread_length" value="${39*itom}" />
+  <xacro:property name="tread_slope_length" value="${11*itom}" />
   <!-- Bin parameters -->
   <!-- Length of top of bin, length of bottom is 13.86 -->

Commit message: Updated the bin model
Note: there is a slight tiny gap at the bottom: this is so small it
really isn't relevant for MoveIt.

File: src/tfr_description/xacro/model_base.xacro (robot description, xacro)
@@ -221,5 +221,5 @@
     </collision>
   </link>
-  <joint name="bin_joint" type="revolute">
+  <joint name="bin_back_joint" type="revolute">
     <parent link="base_link" />
     <child link="bin_back" />

Commit message: Fixed missing tread flap and shifted arm
Shifted the arm on the turntable to its proper position
(may want to verify this again once it's assembled to ensure that
the CAD model is right)

File: src/tfr_description/xacro/model_base.xacro (robot description, xacro)
@@ -205,4 +205,17 @@
     <child link="front_left_slope_link" />
     <origin xyz="${tread_mid_length/2} 0.0 ${tread_mid_height/2}" rpy="0.0 ${(180-160)*dtor} 0.0" />
+  </joint>
+  <link name="front_left_slope_link">
+    <visual>
+      <geometry>
+        <box size="${tread_slope_length} ${tread_width} ${1.25*itom}"/>
+      </geometry>
+      <origin xyz="${tread_slope_length/2} 0.0 ${-1.25/2*itom}" />
+    </visual>
+  </link>
+  <joint name="front_left_slope_joint" type="fixed">
+    <parent link="tread_left_link" />
+    <child link="front_left_slope_link" />
+    <origin xyz="${tread_mid_length/2} 0.0 ${tread_mid_height/2}" rpy="0.0 ${(180-164.1)*dtor} 0.0" />
   </joint>
   <!-- BIN -->

Commit message: Finalized the treads with real dimensions

File: src/tfr_description/xacro/model_base.xacro (robot description, xacro)
@@ -145,5 +145,5 @@
     <parent link="tread_right_link" />
     <child link="front_right_slope_link" />
-    <origin xyz="${tread_mid_length/2} 0.0 ${tread_mid_height/2}" rpy="0.0 ${(180-164.1)*dtor} 0.0" />
+    <origin xyz="${tread_mid_length/2} 0.0 ${tread_mid_height/2}" rpy="0.0 ${(180-160)*dtor} 0.0" />
   </joint>
   <link name="front_left_slope_link">
@@ -158,5 +158,5 @@
     <parent link="tread_left_link" />
     <child link="front_left_slope_link" />
-    <origin xyz="${tread_mid_length/2} 0.0 ${tread_mid_height/2}" rpy="0.0 ${(180-164.1)*dtor} 0.0" />
+    <origin xyz="${tread_mid_length/2} 0.0 ${tread_mid_height/2}" rpy="0.0 ${(180-160)*dtor} 0.0" />
   </joint>
   <!-- BIN -->

File: src/tfr_description/xacro/model_constants.xacro (robot description, xacro)
@@ -15,10 +15,8 @@
   <xacro:property name="drivebase_total_height" value="${6*itom}" />
   <!-- Drivetrain parameters -->
-  <xacro:property name="tread_end_height" value="${11*itom}" />
-  <xacro:property name="tread_end_length" value="${11*itom}" />
-  <xacro:property name="tread_end_radius" value="${(5.5+1.25)*itom}" />
-  <xacro:property name="tread_mid_height" value="${(12.89+(1.25*2))*itom}" />
+  <xacro:property name="tread_end_radius" value="${(13.5/2)*itom}" />
+  <xacro:property name="tread_mid_height" value="${17*itom}" />
   <xacro:property name="tread_mid_length" value="${24*itom}" />
-  <xacro:property name="tread_width" value="${5.75*itom}" />
+  <xacro:property name="tread_width" value="${6*itom}" />
   <xacro:property name="tread_spacing" value="${16*itom}" />
   <xacro:property name="intertread_length" value="${39*itom}" />

Commit message: Finalized the treads with real dimensions

File: src/tfr_description/xacro/model_base.xacro (robot description, xacro)
@@ -217,5 +217,5 @@
     <parent link="tread_left_link" />
     <child link="front_left_slope_link" />
-    <origin xyz="${tread_mid_length/2} 0.0 ${tread_mid_height/2}" rpy="0.0 ${(180-164.1)*dtor} 0.0" />
+    <origin xyz="${tread_mid_length/2} 0.0 ${tread_mid_height/2}" rpy="0.0 ${(180-160)*dtor} 0.0" />
   </joint>
   <!-- BIN -->

Commit message: Updated the arm dimensions based on real measurements.
Next step is to re-add the collision tags I removed.

File: src/tfr_description/xacro/model_base.xacro (robot description, xacro)
@@ -200,17 +200,4 @@
       <origin xyz="${tread_slope_length/2} 0.0 ${-1.25/2*itom}" />
     </collision>
-  </link>
-  <joint name="front_left_slope_joint" type="fixed">
-    <parent link="tread_left_link" />
-    <child link="front_left_slope_link" />
-    <origin xyz="${tread_mid_length/2} 0.0 ${tread_mid_height/2}" rpy="0.0 ${(180-160)*dtor} 0.0" />
-  </joint>
-  <link name="front_left_slope_link">
-    <visual>
-      <geometry>
-        <box size="${tread_slope_length} ${tread_width} ${1.25*itom}"/>
-      </geometry>
-      <origin xyz="${tread_slope_length/2} 0.0 ${-1.25/2*itom}" />
-    </visual>
   </link>
   <joint name="front_left_slope_joint" type="fixed">

Commit message: Got the new model ready for MoveIt

File: src/tfr_description/xacro/model_base.xacro (robot description, xacro)
@@ -221,5 +221,5 @@
     </collision>
   </link>
-  <joint name="bin_back_joint" type="revolute">
+  <joint name="bin_joint" type="revolute">
     <parent link="base_link" />
     <child link="bin_back" />

Commit message: broke potentiometer

File: src/tfr_description/xacro/model_base.xacro (robot description, xacro)
@@ -210,5 +210,5 @@
     <visual>
       <geometry>
-        <box size="${0.125*itom} ${bin_width} ${bin_height}" />
+        <box size="${0.125*itom} ${bin_width} ${bin_back_height}" />
       </geometry>
       <origin xyz="${bin_length} 0 ${-bin_height/2 + bin_height - (9.88 * itom) + (0.5*itom)}" />
@@ -303,5 +303,5 @@
         <box size="${0.125*itom} ${bin_width} ${bin_height*sqrt2}" />
       </geometry>
-      <origin xyz="0.22 0 0"/>
+      <origin xyz="0.17 0 0"/>
     </visual>
     <collision>
@@ -309,5 +309,5 @@
         <box size="${0.125*itom} ${bin_width} ${bin_height*sqrt2}" />
       </geometry>
-      <origin xyz=" 0.22  0 0"/>
+      <origin xyz=" 0.17  0 0"/>
     </collision>
   </link>

File: src/tfr_description/xacro/model_constants.xacro (robot description, xacro)
@@ -25,7 +25,8 @@
   <!-- Length of top of bin, length of bottom is 13.86 -->
   <!-- Using the bigger size as a box instead of making complex angled shape -->
-  <xacro:property name="bin_length" value="${25.78*itom}" />
+  <xacro:property name="bin_length" value="${28.5*itom}" />
   <xacro:property name="bin_width" value="${13.5*itom}" />
-  <xacro:property name="bin_height" value="${15*itom}" />
+  <xacro:property name="bin_height" value="${14*itom}" />
+  <xacro:property name="bin_back_height" value="${10*itom}" />
   <!-- Turntable parameters -->
   <xacro:property name="turntable_radius" value="${4.92*itom}" />
@@ -38,5 +39,5 @@
   <xacro:property name="lower_arm_width" value="${6*itom}" />
   <xacro:property name="lower_arm_height" value="${6*itom}" />
-  <xacro:property name="lower_arm_min" value="0.1045" />
+  <xacro:property name="lower_arm_min" value="0.104" />
   <xacro:property name="lower_arm_max" value="1.35" />
   <!-- Upper arm parameters -->
@@ -44,5 +45,5 @@
   <xacro:property name="upper_arm_width" value="${4.75*itom}" />
   <xacro:property name="upper_arm_height" value="${5*itom}" />
-  <xacro:property name="upper_arm_min" value="1.06465"/>
+  <xacro:property name="upper_arm_min" value="0.98"/>
   <xacro:property name="upper_arm_max" value="2.4"/>
   <!-- Scoop parameters -->
@@ -51,4 +52,4 @@
   <xacro:property name="scoop_diameter" value="${11.2*itom}" />
   <xacro:property name="scoop_min" value="-1.16614" />
-  <xacro:property name="scoop_max" value="1.5937" />
+  <xacro:property name="scoop_max" value="1.62" />
 </robot>
