Commit message: working on navigation

File: src/tfr_description/xacro/model_base.xacro (robot description, xacro)
@@ -303,5 +303,5 @@
         <box size="${0.125*itom} ${bin_width} ${bin_height*sqrt2}" />
       </geometry>
-      <origin xyz="0.17 0 0"/>
+      <origin xyz="0.1 0 0"/>
     </visual>
     <collision>
@@ -309,5 +309,5 @@
         <box size="${0.125*itom} ${bin_width} ${bin_height*sqrt2}" />
       </geometry>
-      <origin xyz=" 0.17  0 0"/>
+      <origin xyz=" 0.1  0 0"/>
     </collision>
   </link>

File: src/tfr_description/xacro/model_constants.xacro (robot description, xacro)
@@ -25,7 +25,7 @@
   <!-- Length of top of bin, length of bottom is 13.86 -->
   <!-- Using the bigger size as a box instead of making complex angled shape -->
-  <xacro:property name="bin_length" value="${28.5*itom}" />
+  <xacro:property name="bin_length" value="${29.5*itom}" />
   <xacro:property name="bin_width" value="${13.5*itom}" />
-  <xacro:property name="bin_height" value="${14*itom}" />
+  <xacro:property name="bin_height" value="${11.5*itom}" />
   <xacro:property name="bin_back_height" value="${10*itom}" />
   <!-- Turntable parameters -->
@@ -40,5 +40,5 @@
   <xacro:property name="lower_arm_height" value="${6*itom}" />
   <xacro:property name="lower_arm_min" value="0.104" />
-  <xacro:property name="lower_arm_max" value="1.35" />
+  <xacro:property name="lower_arm_max" value="1.55" />
   <!-- Upper arm parameters -->
   <xacro:property name="upper_arm_length" value="${20*itom}" />
@@ -49,6 +49,6 @@
   <!-- Scoop parameters -->
   <xacro:property name="scoop_width" value="${8.5*itom}" />
-  <xacro:property name="scoop_length" value="${10*itom}" />
-  <xacro:property name="scoop_diameter" value="${11.2*itom}" />
+  <xacro:property name="scoop_length" value="${11.75*itom}" />
+  <xacro:property name="scoop_diameter" value="${10.5*itom}" />
   <xacro:property name="scoop_min" value="-1.16614" />
   <xacro:property name="scoop_max" value="1.62" />

Commit message: refined digging cycle

File: src/tfr_description/xacro/model_base.xacro (robot description, xacro)
@@ -303,5 +303,5 @@
         <box size="${0.125*itom} ${bin_width} ${bin_height*sqrt2}" />
       </geometry>
-      <origin xyz="0.1 0 0"/>
+      <origin xyz="${bin_back_offset} 0 0"/>
     </visual>
     <collision>
@@ -309,5 +309,5 @@
         <box size="${0.125*itom} ${bin_width} ${bin_height*sqrt2}" />
       </geometry>
-      <origin xyz=" 0.1  0 0"/>
+      <origin xyz=" ${bin_back_offset}  0 0"/>
     </collision>
   </link>

File: src/tfr_description/xacro/model_constants.xacro (robot description, xacro)
@@ -25,8 +25,9 @@
   <!-- Length of top of bin, length of bottom is 13.86 -->
   <!-- Using the bigger size as a box instead of making complex angled shape -->
-  <xacro:property name="bin_length" value="${29.5*itom}" />
+  <xacro:property name="bin_length" value="${33*itom}" />
   <xacro:property name="bin_width" value="${13.5*itom}" />
-  <xacro:property name="bin_height" value="${12.5*itom}" />
-  <xacro:property name="bin_back_height" value="${10*itom}" />
+  <xacro:property name="bin_height" value="${13*itom}" />
+  <xacro:property name="bin_back_height" value="${8*itom}" />
+  <xacro:property name="bin_back_offset" value="${6.5*itom}" />
   <!-- Turntable parameters -->
   <xacro:property name="turntable_radius" value="${4.92*itom}" />
@@ -49,6 +50,6 @@
   <!-- Scoop parameters -->
   <xacro:property name="scoop_width" value="${8.5*itom}" />
-  <xacro:property name="scoop_length" value="${12.5*itom}" />
-  <xacro:property name="scoop_diameter" value="${10*itom}" />
+  <xacro:property name="scoop_length" value="${13.5*itom}" />
+  <xacro:property name="scoop_diameter" value="${11.5*itom}" />
   <xacro:property name="scoop_min" value="-1.16614" />
   <xacro:property name="scoop_max" value="1.62" />
