Commit message: added arm control, ready for pid tuning

File: src/tfr_description/xacro/model_constants.xacro (robot description, xacro)
@@ -38,16 +38,16 @@
   <xacro:property name="lower_arm_width" value="${4*itom}" />
   <xacro:property name="lower_arm_height" value="${6*itom}" />
-  <xacro:property name="lower_arm_min" value="${5.5*dtor}" />
-  <xacro:property name="lower_arm_max" value="${85*dtor}" /> <!-- TODO: must be determined once mounted-->
+  <xacro:property name="lower_arm_min" value="0.07" />
+  <xacro:property name="lower_arm_max" value="1.5" />
   <!-- Upper arm parameters -->
   <xacro:property name="upper_arm_length" value="${20*itom}" />
   <xacro:property name="upper_arm_width" value="${3.625*itom}" />
   <xacro:property name="upper_arm_height" value="${5*itom}" />
-  <xacro:property name="upper_arm_min" value="${48*dtor}" />
-  <xacro:property name="upper_arm_max" value="${113*dtor}" />
+  <xacro:property name="upper_arm_min" value="0.998" />
+  <xacro:property name="upper_arm_max" value="2.21" />
   <!-- Scoop parameters -->
   <xacro:property name="scoop_width" value="${10*itom}" />
   <xacro:property name="scoop_diameter" value="${10.5*itom}" />
-  <xacro:property name="scoop_min" value="${-61*dtor}" />
-  <xacro:property name="scoop_max" value="${78*dtor}" />
+  <xacro:property name="scoop_min" value="-1.607" />
+  <xacro:property name="scoop_max" value="1.15" />
 </robot>

Commit message: tested all 3 jointsy

File: src/tfr_description/xacro/model_constants.xacro (robot description, xacro)
@@ -47,7 +47,7 @@
   <xacro:property name="upper_arm_max" value="2.21" />
   <!-- Scoop parameters -->
-  <xacro:property name="scoop_width" value="${10*itom}" />
-  <xacro:property name="scoop_diameter" value="${10.5*itom}" />
-  <xacro:property name="scoop_min" value="-1.607" />
-  <xacro:property name="scoop_max" value="1.15" />
+  <xacro:property name="scoop_width" value="${10.25*itom}" />
+  <xacro:property name="scoop_diameter" value="${11.5*itom}" />
+  <xacro:property name="scoop_min" value="-1.633" />
+  <xacro:property name="scoop_max" value="1.115" />
 </robot>

Commit message: integrated one mining motion

File: src/tfr_description/xacro/model_constants.xacro (robot description, xacro)
@@ -38,5 +38,5 @@
   <xacro:property name="lower_arm_width" value="${4*itom}" />
   <xacro:property name="lower_arm_height" value="${6*itom}" />
-  <xacro:property name="lower_arm_min" value="0.07" />
+  <xacro:property name="lower_arm_min" value="0.034" />
   <xacro:property name="lower_arm_max" value="1.5" />
   <!-- Upper arm parameters -->
@@ -44,10 +44,10 @@
   <xacro:property name="upper_arm_width" value="${3.625*itom}" />
   <xacro:property name="upper_arm_height" value="${5*itom}" />
-  <xacro:property name="upper_arm_min" value="0.998" />
-  <xacro:property name="upper_arm_max" value="2.21" />
+  <xacro:property name="upper_arm_min" value="0.92" />
+  <xacro:property name="upper_arm_max" value="2.16" />
   <!-- Scoop parameters -->
   <xacro:property name="scoop_width" value="${10.25*itom}" />
   <xacro:property name="scoop_diameter" value="${11.5*itom}" />
-  <xacro:property name="scoop_min" value="-1.633" />
-  <xacro:property name="scoop_max" value="1.115" />
+  <xacro:property name="scoop_min" value="-1.67" />
+  <xacro:property name="scoop_max" value="1.07" />
 </robot>

Commit message: added control safety for arm reset

File: src/tfr_description/xacro/model_constants.xacro (robot description, xacro)
@@ -26,11 +26,11 @@
   <!-- Using the bigger size as a box instead of making complex angled shape -->
   <xacro:property name="bin_length" value="${25.78*itom}" />
-  <xacro:property name="bin_width" value="${11*itom}" />
-  <xacro:property name="bin_height" value="${11.5*itom}" />
+  <xacro:property name="bin_width" value="${10.5*itom}" />
+  <xacro:property name="bin_height" value="${13*itom}" />
   <!-- Turntable parameters -->
   <xacro:property name="turntable_radius" value="${4.92*itom}" />
   <!-- 1" in model plus undefined height for mounting and extra components -->
   <!-- Rounded to 2" for now -->
-  <xacro:property name="turntable_height" value="${1.2*itom}" />
+  <xacro:property name="turntable_height" value="${2.25*itom}" />
   <!-- Lower arm parameters -->
   <xacro:property name="lower_arm_length" value="${22*itom}" />
@@ -38,16 +38,16 @@
   <xacro:property name="lower_arm_width" value="${4*itom}" />
   <xacro:property name="lower_arm_height" value="${6*itom}" />
-  <xacro:property name="lower_arm_min" value="0.034" />
-  <xacro:property name="lower_arm_max" value="1.5" />
+  <xacro:property name="lower_arm_min" value="0.1048" />
+  <xacro:property name="lower_arm_max" value="1.63" />
   <!-- Upper arm parameters -->
   <xacro:property name="upper_arm_length" value="${20*itom}" />
   <xacro:property name="upper_arm_width" value="${3.625*itom}" />
   <xacro:property name="upper_arm_height" value="${5*itom}" />
-  <xacro:property name="upper_arm_min" value="0.92" />
-  <xacro:property name="upper_arm_max" value="2.16" />
+  <xacro:property name="upper_arm_min" value="1.06465"/>
+  <xacro:property name="upper_arm_max" value="2.295108" />
   <!-- Scoop parameters -->
-  <xacro:property name="scoop_width" value="${10.25*itom}" />
+  <xacro:property name="scoop_width" value="${10.2*itom}" />
   <xacro:property name="scoop_diameter" value="${11.5*itom}" />
-  <xacro:property name="scoop_min" value="-1.67" />
-  <xacro:property name="scoop_max" value="1.07" />
+  <xacro:property name="scoop_min" value="-1.41372" />
+  <xacro:property name="scoop_max" value="1.48353" />
 </robot>

Commit message: did field testy

File: src/tfr_description/xacro/model_constants.xacro (robot description, xacro)
@@ -47,6 +47,6 @@
   <xacro:property name="upper_arm_max" value="2.295108" />
   <!-- Scoop parameters -->
-  <xacro:property name="scoop_width" value="${10.2*itom}" />
-  <xacro:property name="scoop_diameter" value="${11.5*itom}" />
+  <xacro:property name="scoop_width" value="${10*itom}" />
+  <xacro:property name="scoop_diameter" value="${10*itom}" />
   <xacro:property name="scoop_min" value="-1.41372" />
   <xacro:property name="scoop_max" value="1.48353" />

Commit message: working on digging procedure fixing drivebase odom

File: src/tfr_description/xacro/model_constants.xacro (robot description, xacro)
@@ -27,5 +27,5 @@
   <xacro:property name="bin_length" value="${29.5*itom}" />
   <xacro:property name="bin_width" value="${13.5*itom}" />
-  <xacro:property name="bin_height" value="${11.5*itom}" />
+  <xacro:property name="bin_height" value="${12.5*itom}" />
   <xacro:property name="bin_back_height" value="${10*itom}" />
   <!-- Turntable parameters -->

Commit message: integrated bin

File: src/tfr_description/xacro/model_constants.xacro (robot description, xacro)
@@ -49,6 +49,6 @@
   <!-- Scoop parameters -->
   <xacro:property name="scoop_width" value="${8.5*itom}" />
-  <xacro:property name="scoop_length" value="${11.75*itom}" />
-  <xacro:property name="scoop_diameter" value="${10.5*itom}" />
+  <xacro:property name="scoop_length" value="${12.5*itom}" />
+  <xacro:property name="scoop_diameter" value="${10*itom}" />
   <xacro:property name="scoop_min" value="-1.16614" />
   <xacro:property name="scoop_max" value="1.62" />

Commit message: integration testing/mining refinement

File: src/tfr_description/xacro/model_constants.xacro (robot description, xacro)
@@ -25,8 +25,8 @@
   <!-- Length of top of bin, length of bottom is 13.86 -->
   <!-- Using the bigger size as a box instead of making complex angled shape -->
-  <xacro:property name="bin_length" value="${33*itom}" />
+  <xacro:property name="bin_length" value="${36*itom}" />
   <xacro:property name="bin_width" value="${13.5*itom}" />
-  <xacro:property name="bin_height" value="${13*itom}" />
-  <xacro:property name="bin_back_height" value="${8*itom}" />
+  <xacro:property name="bin_height" value="${16*itom}" />
+  <xacro:property name="bin_back_height" value="${9*itom}" />
   <xacro:property name="bin_back_offset" value="${6.5*itom}" />
   <!-- Turntable parameters -->
@@ -50,6 +50,6 @@
   <!-- Scoop parameters -->
   <xacro:property name="scoop_width" value="${8.5*itom}" />
-  <xacro:property name="scoop_length" value="${13.5*itom}" />
-  <xacro:property name="scoop_diameter" value="${11.5*itom}" />
+  <xacro:property name="scoop_length" value="${12*itom}" />
+  <xacro:property name="scoop_diameter" value="${12.5*itom}" />
   <xacro:property name="scoop_min" value="-1.16614" />
   <xacro:property name="scoop_max" value="1.62" />
